Commit message: Add urdf link collision and inertia

File: src/swarm/models/robot.urdf (robot description, URDF)
Before this commit: robot my_robot, 3 links, 2 joints
Links:
- link chassis: mass None -> 10; geometry collision box size=1 0.5 0.1; visual box size=1 0.5 0.1
- link left_wheel: mass None -> 4; geometry collision cylinder length=0.1 radius=0.3; visual cylinder length=0.1 radius=0.3
- link right_wheel: mass None -> 4; geometry collision cylinder length=0.1 radius=0.3; visual cylinder length=0.1 radius=0.3

Commit message: Add a caster wheel to robot for stability

File: src/swarm/models/robot.urdf (robot description, URDF)
Before this commit: robot my_robot, 3 links, 2 joints
Links:
- added link caster_wheel, mass 1; collision sphere radius=0.15; visual sphere radius=0.15
Joints:
- added joint caster_wheel_to_chassis: type continuous, parent chassis, child caster_wheel, origin xyz=0 0 -0.15 rpy=0 0 0, axis 0 1 0

Commit message: Add a dummy base_link to serve as the root link of the urdf
This is added because the root link is required to not have inertial
properties, hence the chassis link cannot be the root link

File: src/swarm/models/robot.urdf (robot description, URDF)
Before this commit: robot my_robot, 4 links, 3 joints
Links:
- added link base_link
Joints:
- added joint chassis_to_base_link: type fixed, parent base_link, child chassis

Commit message: Align robot wheels

File: src/swarm/models/robot.urdf (robot description, URDF)
Before this commit: robot my_robot, 5 links, 4 joints
Links:
- link caster_wheel: geometry collision sphere radius=0.125; visual sphere radius=0.125
Joints:
- joint caster_wheel_to_chassis: origin xyz=0 0 -0.15 rpy=0 0 0 -> xyz=0.35 0 -0.175 rpy=0 0 0
- joint left_wheel_to_chassis: origin (none) -> xyz=-0.2 0 0 rpy=0 0 0
- joint right_wheel_to_chassis: origin (none) -> xyz=-0.2 0 0 rpy=0 0 0

Commit message: Add a camera to the robot urdf

File: src/swarm/models/robot.urdf (robot description, URDF)
Before this commit: robot my_robot, 5 links, 4 joints
Links:
- added link camera_link; collision box size=0.1 0.1 0.1; visual box size=0.1 0.1 0.1
Joints:
- added joint camera_to_chassis: type fixed, parent chassis, child camera_link, origin xyz=0.4 0 0.1 rpy=0 0 0

Commit message: Add lidar sensor to robot

File: src/swarm/models/robot.urdf (robot description, URDF)
Before this commit: robot my_robot, 6 links, 5 joints
Links:
- added link lidar_link; visual cylinder length=0.2 radius=0.1
Joints:
- added joint lidar_joint: type fixed, parent chassis, child lidar_link, origin xyz=0 0 0.1 rpy=0 0 0
