Commit message: Fix camera feed showing shadows on rviz2
Camera was facing upwards in rviz hence showing some parts of the
robots chassis and the lidar above. This happened because rviz and
gazebo use different camera feed coordinate frames. Fixed by creating
a camera optical link, attaching the camera feed to it and rotating it
to face forward

File: src/swarm/models/rover.xacro (robot description, xacro)
@@ -16,5 +16,6 @@
     <xacro:property name="wheel_mass" value="2"/>
     <xacro:property name="chassis_mass" value="10"/>
-    <xacro:property name="camera_size" value="0.01"/>
+    <xacro:property name="camera_size" value="0.03"/>
+    <xacro:property name="camera_thickness" value="0.01"/>
     <xacro:property name="lidar_size" value="0.1"/>
     <!-- macros -->
@@ -89,5 +90,5 @@
         <visual>
             <geometry>
-                <box size="${camera_size} ${camera_size} ${camera_size}"/>
+                <box size="${camera_thickness} ${camera_size} ${camera_size}"/>
             </geometry>
             <material name="black"/>
@@ -95,9 +96,10 @@
         <collision>
             <geometry>
-                <box size="${camera_size} ${camera_size} ${camera_size}"/>
+                <box size="${camera_thickness} ${camera_size} ${camera_size}"/>
             </geometry>
-            <xacro:box_inertia mass="0.001" l="${camera_size}" w="${camera_size}" h="${camera_size}"/>
+            <xacro:box_inertia mass="0.001" l="${camera_thickness}" w="${camera_size}" h="${camera_size}"/>
         </collision>
     </link>
+    <link name="camera_link_optical" />
     <link name="lidar_link">
         <visual>
@@ -126,5 +128,10 @@
         <parent link="chassis"/>
         <child link="camera_link"/>
-        <origin rpy="0.0 0.0 0.0" xyz="${chassis_length/2 + camera_size/2} 0.0 0.0"/>
+        <origin rpy="0.0 0.0 0.0" xyz="${chassis_length/2 + camera_thickness} 0.0 ${chassis_height/4}"/>
+    </joint>
+    <joint name="camera_link_optical_joint" type="fixed">
+        <parent link="camera_link"/>
+        <child link="camera_link_optical"/>
+        <origin rpy="${-pi/2} 0.0 ${-pi/2}" xyz="${camera_thickness} 0.0 0.0"/>
     </joint>
     <joint name="lidar_link_joint" type="fixed">
@@ -133,5 +140,4 @@
         <origin rpy="0.0 0.0 0.0" xyz="${chassis_length/2 - 0.15} 0.0 ${chassis_height/2 + lidar_size/2}"/>
     </joint>
-    <!-- gazebo plugins -->
     <!-- wheels friction -->
     <xacro:friction_coefficients link_name="rear_left_wheel" />
@@ -139,4 +145,5 @@
     <xacro:friction_coefficients link_name="front_left_wheel" />
     <xacro:friction_coefficients link_name="front_right_wheel" />
+    <!-- gazebo plugins -->
     <xacro:include filename="$(find swarm)/models/rover.gazebo" />
 </robot>

Commit message: Add imu sensor to robot
I want to use the imu sensor for localization by fusing it with
the diff drive odometry data.

File: src/swarm/models/rover.xacro (robot description, xacro)
@@ -19,4 +19,5 @@
     <xacro:property name="camera_thickness" value="0.01"/>
     <xacro:property name="lidar_size" value="0.1"/>
+    <xacro:property name="odometry_update_rate" value="5"/>
     <!-- macros -->
     <xacro:macro name="box_inertia" params="mass l w h">
