Commit message: Configure ekf_node from the robot_localization package for 2D localisation

File: src/swarm/models/rover/rover.xacro (robot description, xacro)
@@ -21,5 +21,5 @@
     <xacro:property name="camera_thickness" value="0.01"/>
     <xacro:property name="lidar_size" value="0.1"/>
-    <xacro:property name="odometry_update_rate" value="5"/>
+    <xacro:property name="odometry_update_rate" value="30"/>
     <!-- macros -->
     <xacro:macro name="box_inertia" params="mass l w h">
